File: sab_v4_mini/sab_v4_mini.kicad_pcb (KiCad board)
At the start: 4 copper layers, 265 x 117 mm, 404 parts, among them J1 External_POT, J11 AudioJack_LOOP3_SEND, J12 AudioJack_LOOP3_RETURN, J13 AudioJack_OUTPUT, J14 AudioJack_INPUT, J15 AudioJack_LOOP2_RETURN, J16 STlink_DISP_MCU, J17 Conn_01x10_Footswitch, J18 Conn_01x16_ILI9341, J2 STlink_DSP, J3 Barrel_Jack_Switch, J4 Conn_01x02_i2c, J5 USB_C_Receptacle_USB2.0, J7 AudioJack_LOOP1_SEND, J8 AudioJack_LOOP1_RETURN, J9 AudioJack_LOOP2_SEND, SW1 SW_SPST, SW2 SW_SPST, U1 IS42S16100H-7TL, U10 OP275, U12 OP275, U13 74HC14, U14 OP275, U15 STM32H723ZGTx, U16 USBLC6-2P6, U17 W25Q128JVS, U18 W25Q128JVS, U19 FE1.1s, U2 OP275, U20 AP1117-33, U3 7909, U4 OP275, U5 AP1117-33, U6 7809, U7 STM32H723ZGTx, U8 OP275, U9 AP1117-33, Y1 X1E0000210132, Y2 X1E0000210132, Y3 Crystal_GND24

Commit message: added codec
Parts:
- removed C121, C122: 2.2uF, Capacitor_SMD:C_0805_2012Metric_Pad1.18x1.45mm_HandSolder
- removed C123, C125: 12pF, Capacitor_SMD:C_0603_1608Metric
- removed C124, C126, C127, C128, C129, C130, C131, C185, C186, C187, C188, C189, C221, C227, C79: 100nF, Capacitor_SMD:C_0603_1608Metric
- removed C203, C204: 20pF, Capacitor_SMD:C_0402_1005Metric
- removed C218, C219, C223, C224, C225, C226: 10uF, Capacitor_SMD:C_1206_3216Metric
- removed C220, C222: 100uF, stm_audio_board_footprints:CP_Radial_D6.3mm_P2.50mm_reference_fix
- removed C228, C68: 1nF, Capacitor_SMD:C_0603_1608Metric
- removed C26: 100uF tantal, Capacitor_Tantalum_SMD:CP_EIA-3528-21_Kemet-B
- removed C67: 33nF, Capacitor_SMD:C_0805_2012Metric_Pad1.18x1.45mm_HandSolder
- removed C80: 10uF tantal, Capacitor_Tantalum_SMD:CP_EIA-3216-18_Kemet-A
- removed DISPLAY_OK1: LED, LED_SMD:LED_0603_1608Metric_Pad1.05x0.95mm_HandSolder
- removed J1: External_POT, stm_audio_board_footprints:6.3_jack_new_ref
- removed J17: Conn_01x10_Footswitch, Connector_IDC:IDC-Header_2x05_P2.54mm_Vertical
- removed J18: Conn_01x16_ILI9341, Connector_PinHeader_2.54mm:PinHeader_1x16_P2.54mm_Vertical
- removed R1, R18, R75, R78, R80, R82: 10k, Resistor_SMD:R_0603_1608Metric
- removed R10: 3k, Resistor_SMD:R_0603_1608Metric
- removed R24, R74: 100R, Resistor_SMD:R_0603_1608Metric
- removed R33, R76, R77, R79, R81, R83, R84, R85: 1k, Resistor_SMD:R_0603_1608Metric
- removed R87: 2.7k, Resistor_SMD:R_0603_1608Metric
- removed RV1, RV2, RV3, RV4, RV5, RV6: R_Potentiometer, Potentiometer_THT:Potentiometer_Alps_RK09L_Single_Vertical
- removed SW2: SW_SPST, Button_Switch_SMD:SW_SPST_TL3305A
- removed TP7: TestPoint_3V3, TestPoint:TestPoint_Pad_D1.5mm
- removed U13: 74HC14, Package_SO:SOIC-14_3.9x8.7mm_P1.27mm
- removed U15: STM32H723ZGTx, Package_QFP:LQFP-144_20x20mm_P0.5mm
- removed U17, U18: W25Q128JVS, Package_SO:SOIC-8_5.23x5.23mm_P1.27mm
- removed U19: FE1.1s, Package_SO:SSOP-28_3.9x9.9mm_P0.635mm
- removed Y1: X1E0000210132, Crystal:Crystal_SMD_SeikoEpson_TSX3225-4Pin_3.2x2.5mm_HandSoldering
- removed Y3: Crystal_GND24, Crystal:Crystal_SMD_3225-4Pin_3.2x2.5mm
- added C25: 100nF, Capacitor_SMD:C_0603_1608Metric, F.Cu at (22.0, 10.1)
- added R12: 10k, Resistor_SMD:R_0603_1608Metric, F.Cu at (1.50, 19.2)
- added U7: STM32H750VBTx, Package_QFP:LQFP-100_14x14mm_P0.5mm, F.Cu at (8.74, 8.74)
- added U9: CS4270, Package_SO:TSSOP-24_4.4x7.8mm_P0.65mm, F.Cu at (24.7, 4.17)
- R12: value 1k -> 10k
- U7: value STM32H723ZGTx -> STM32H750VBTx; footprint Package_QFP:LQFP-144_20x20mm_P0.5mm -> Package_QFP:LQFP-100_14x14mm_P0.5mm
- U9: value AP1117-33 -> CS4270; footprint Package_TO_SOT_SMD:SOT-223 -> Package_SO:TSSOP-24_4.4x7.8mm_P0.65mm
Connections:
- net Net-(U19-VBUSM) renamed DSP_VBUS
- C1 pad 2: GND -> Audio_Loop3_Return
- C10 pad 2: GND -> Audio_Loop3_Return
- C101 pad 1: GND -> Audio_Loop3_Return
- C102 pad 2: GND -> Audio_Loop3_Return
- C106 pad 2: GND -> Audio_Loop3_Return
- C108 pad 1: GND -> Audio_Loop3_Return
- C109 pad 2: GND -> Audio_Loop3_Return
- C11 pad 2: GND -> Audio_Loop3_Return
- C111 pad 1: GND -> Audio_Loop3_Return
- C113 pad 2: GND -> Audio_Loop3_Return
- C114 pad 1: GND -> Audio_Loop3_Return
- C115 pad 2: GND -> Audio_Loop3_Return
- C117 pad 1: GND -> Audio_Loop3_Return
- C119 pad 2: GND -> Audio_Loop3_Return
- C12 pad 2: GND -> Audio_Loop3_Return
- C120 pad 2: GND -> Audio_Loop3_Return
- C134 pad 2: GND -> Audio_Loop3_Return
- C135 pad 1: GND -> Audio_Loop3_Return
- C139 pad 2: GND -> Audio_Loop3_Return
- C14 pad 2: GND -> Audio_Loop3_Return
- C140 pad 2: GND -> Audio_Loop3_Return
- C141 pad 2: GND -> Audio_Loop3_Return
- C142 pad 2: GND -> Audio_Loop3_Return
- C143 pad 2: GND -> Audio_Loop3_Return
- C144 pad 2: GND -> Audio_Loop3_Return
- C145 pad 2: GND -> Audio_Loop3_Return
- C146 pad 2: GND -> Audio_Loop3_Return
- C147 pad 2: GND -> Audio_Loop3_Return
- C148 pad 2: GND -> Audio_Loop3_Return
- C149 pad 2: GND -> Audio_Loop3_Return
- C15 pad 2: GND -> Audio_Loop3_Return
- C150 pad 2: GND -> Audio_Loop3_Return
- C151 pad 2: GND -> Audio_Loop3_Return
- C152 pad 2: GND -> Audio_Loop3_Return
- C153 pad 2: GND -> Audio_Loop3_Return
- C154 pad 2: GND -> Audio_Loop3_Return
- C155 pad 2: GND -> Audio_Loop3_Return
- C157 pad 2: GND -> Audio_Loop3_Return
- C158 pad 2: GND -> Audio_Loop3_Return
- C16 pad 1: /MCU/NRST -> NRST
- C16 pad 2: GND -> Audio_Loop3_Return
- C160 pad 2: GND -> Audio_Loop3_Return
- C161 pad 2: GND -> Audio_Loop3_Return
- C163 pad 2: GND -> Audio_Loop3_Return
- C164 pad 2: GND -> Audio_Loop3_Return
- C165 pad 2: GND -> Audio_Loop3_Return
- C166 pad 2: GND -> Audio_Loop3_Return
- C167 pad 2: GND -> Audio_Loop3_Return
- C168 pad 2: GND -> Audio_Loop3_Return
- C169 pad 2: GND -> Audio_Loop3_Return
- C17 pad 2: GND -> Audio_Loop3_Return
- C170 pad 2: GND -> Audio_Loop3_Return
- C171 pad 2: GND -> Audio_Loop3_Return
- C172 pad 2: GND -> Audio_Loop3_Return
- C173 pad 2: GND -> Audio_Loop3_Return
- C174 pad 1: GND -> Audio_Loop3_Return
- C175 pad 1: GND -> Audio_Loop3_Return
- C176 pad 1: GND -> Audio_Loop3_Return
- C177 pad 1: GND -> Audio_Loop3_Return
- C178 pad 1: GND -> Audio_Loop3_Return
- C179 pad 2: GND -> Audio_Loop3_Return
- C18 pad 2: GND -> Audio_Loop3_Return
- C180 pad 1: GND -> Audio_Loop3_Return
- C181 pad 2: GND -> Audio_Loop3_Return
- C182 pad 2: GND -> Audio_Loop3_Return
- C183 pad 2: GND -> Audio_Loop3_Return
- C184 pad 2: GND -> Audio_Loop3_Return
- C19 pad 1: GND -> Audio_Loop3_Return
- C190 pad 2: GND -> Audio_Loop3_Return
- C191 pad 2: GND -> Audio_Loop3_Return
- C192 pad 2: GND -> Audio_Loop3_Return
- C193 pad 2: GND -> Audio_Loop3_Return
- C194 pad 2: GND -> Audio_Loop3_Return
- C195 pad 2: GND -> Audio_Loop3_Return
- C196 pad 2: GND -> Audio_Loop3_Return
- C197 pad 2: GND -> Audio_Loop3_Return
- C198 pad 2: GND -> Audio_Loop3_Return
- C199 pad 2: GND -> Audio_Loop3_Return
- C2 pad 1: GND -> Audio_Loop3_Return
- C200 pad 2: GND -> Audio_Loop3_Return
- C201 pad 2: GND -> Audio_Loop3_Return
- C202 pad 2: GND -> Audio_Loop3_Return
- C205 pad 2: GND -> Audio_Loop3_Return
- C206 pad 2: GND -> Audio_Loop3_Return
- C207 pad 2: GND -> Audio_Loop3_Return
- C208 pad 2: GND -> Audio_Loop3_Return
- C209 pad 2: GND -> Audio_Loop3_Return
- C210 pad 2: GND -> Audio_Loop3_Return
- C211 pad 2: GND -> Audio_Loop3_Return
- C212 pad 2: GND -> Audio_Loop3_Return
- C213 pad 2: GND -> Audio_Loop3_Return
- C214 pad 2: GND -> Audio_Loop3_Return
- C215 pad 2: GND -> Audio_Loop3_Return
- C216 pad 2: GND -> Audio_Loop3_Return
- C217 pad 2: GND -> Audio_Loop3_Return
- C22 pad 1: GND -> Audio_Loop3_Return
- C229 pad 2: GND -> Audio_Loop3_Return
- C23 pad 2: GND -> Audio_Loop3_Return
- C24 pad 1: GND -> Audio_Loop3_Return
- C25 pad 1: GND -> unconnected-(C25-Pad1)
- C25 pad 2: AD1939_CM -> unconnected-(C25-Pad2)
- C27 pad 1: GND -> Audio_Loop3_Return
- C28 pad 2: GND -> Audio_Loop3_Return
- C29 pad 2: GND -> Audio_Loop3_Return
- C3 pad 2: GND -> Audio_Loop3_Return
- C30 pad 2: GND -> Audio_Loop3_Return
- C31 pad 1: GND -> Audio_Loop3_Return
- C32 pad 2: GND -> Audio_Loop3_Return
- C33 pad 2: GND -> Audio_Loop3_Return
- C34 pad 2: GND -> Audio_Loop3_Return
- C35 pad 2: GND -> Audio_Loop3_Return
- C36 pad 2: GND -> Audio_Loop3_Return
- C37 pad 1: GND -> Audio_Loop3_Return
- C38 pad 1: GND -> Audio_Loop3_Return
- C4 pad 2: GND -> Audio_Loop3_Return
- C40 pad 1: GND -> Audio_Loop3_Return
- C41 pad 2: GND -> Audio_Loop3_Return
- C43 pad 2: GND -> Audio_Loop3_Return
- C45 pad 1: GND -> Audio_Loop3_Return
- C47 pad 2: GND -> Audio_Loop3_Return
- C49 pad 2: GND -> Audio_Loop3_Return
- C5 pad 2: GND -> Audio_Loop3_Return
- C50 pad 2: GND -> Audio_Loop3_Return
- C53 pad 2: GND -> Audio_Loop3_Return
- C54 pad 2: GND -> Audio_Loop3_Return
- C55 pad 2: GND -> Audio_Loop3_Return
- C56 pad 2: GND -> Audio_Loop3_Return
- C57 pad 2: GND -> Audio_Loop3_Return
- C58 pad 2: GND -> Audio_Loop3_Return
- C59 pad 2: GND -> Audio_Loop3_Return
- C6 pad 2: GND -> Audio_Loop3_Return
- C60 pad 2: GND -> Audio_Loop3_Return
- C61 pad 2: GND -> Audio_Loop3_Return
- C62 pad 2: GND -> Audio_Loop3_Return
- C63 pad 2: GND -> Audio_Loop3_Return
- C64 pad 2: GND -> Audio_Loop3_Return
- C66 pad 2: GND -> Audio_Loop3_Return
- C7 pad 2: GND -> Audio_Loop3_Return
- C70 pad 2: GND -> Audio_Loop3_Return
- C71 pad 2: GND -> Audio_Loop3_Return
- C74 pad 1: GND -> Audio_Loop3_Return
- C78 pad 2: GND -> Audio_Loop3_Return
- C8 pad 2: GND -> Audio_Loop3_Return
- C81 pad 2: GND -> Audio_Loop3_Return
- C82 pad 2: GND -> Audio_Loop3_Return
- C84 pad 1: GND -> Audio_Loop3_Return
- C86 pad 2: GND -> Audio_Loop3_Return
- C88 pad 2: GND -> Audio_Loop3_Return
- C89 pad 2: GND -> Audio_Loop3_Return
- C9 pad 2: GND -> Audio_Loop3_Return
- C90 pad 2: GND -> Audio_Loop3_Return
- C92 pad 1: GND -> Audio_Loop3_Return
- C93 pad 2: GND -> Audio_Loop3_Return
- C95 pad 1: GND -> Audio_Loop3_Return
- C97 pad 2: GND -> Audio_Loop3_Return
- C99 pad 2: GND -> Audio_Loop3_Return
- D1 pad 2: GND -> Audio_Loop3_Return
- D12 pad 2: GND -> Audio_Loop3_Return
- D14 pad 2: GND -> Audio_Loop3_Return
- D16 pad 2: GND -> Audio_Loop3_Return
- D18 pad 2: GND -> Audio_Loop3_Return
- D20 pad 2: GND -> Audio_Loop3_Return
- D6 pad 2: GND -> Audio_Loop3_Return
- D8 pad 2: GND -> Audio_Loop3_Return
- DSP_OK1 pad 1: GND -> Audio_Loop3_Return
- H1 pad 1: GND -> Audio_Loop3_Return
- H2 pad 1: GND -> Audio_Loop3_Return
- H3 pad 1: GND -> Audio_Loop3_Return
- H4 pad 1: GND -> Audio_Loop3_Return
- H5 pad 1: GND -> Audio_Loop3_Return
- H6 pad 1: GND -> Audio_Loop3_Return
- J12 pad TN: GND -> Audio_Loop3_Return
- J14 pad TN: GND -> Audio_Loop3_Return
- J15 pad TN: GND -> Audio_Loop3_Return
- J16 pad 1: GND -> Audio_Loop3_Return
- J2 pad 1: GND -> Audio_Loop3_Return
- J5 pad A1: GND -> Audio_Loop3_Return
- J5 pad A12: GND -> Audio_Loop3_Return
- J5 pad B1: GND -> Audio_Loop3_Return
- J5 pad B12: GND -> Audio_Loop3_Return
- J8 pad TN: GND -> Audio_Loop3_Return
- PS1 pad 7: GND -> Audio_Loop3_Return
- PS2 pad 7: GND -> Audio_Loop3_Return
- R11 pad 2: AD1939_CM -> VBIAS
- R12 pad 1: Net-(DISPLAY_OK1-A) -> to_BOOT0
- R12 pad 2: DISPLAY_OK_LED -> Net-(J6-Pin_2)
- R20 pad 1: GND -> Audio_Loop3_Return
- R3 pad 2: AD1939_CM -> VBIAS
- R32 pad 1: GND -> Audio_Loop3_Return
- R34 pad 2: AD1939_CM -> VBIAS
- R37 pad 2: AD1939_CM -> VBIAS
- R43 pad 2: AD1939_CM -> VBIAS
- R46 pad 2: AD1939_CM -> VBIAS
- R52 pad 2: AD1939_CM -> VBIAS
- R55 pad 2: AD1939_CM -> VBIAS
- R62 pad 1: GND -> Audio_Loop3_Return
- R70 pad 1: GND -> Audio_Loop3_Return
- SW1 pad 1: /MCU/NRST -> NRST
- SW1 pad 2: GND -> Audio_Loop3_Return
- U1 pad 10: GND -> Audio_Loop3_Return
- U1 pad 11: /MCU/DSP_SDRAM_DATA_BUS6 -> (no net)
- U1 pad 12: /MCU/DSP_SDRAM_DATA_BUS7 -> (no net)
- U1 pad 14: /MCU/DSP_SDRAM_LDQM -> (no net)
- U1 pad 15: /MCU/DSP_SDRAM_WE -> (no net)
- U1 pad 16: /MCU/DSP_SDRAM_CAS -> (no net)
- U1 pad 17: /MCU/DSP_SDRAM_RAS -> (no net)
- U1 pad 18: /MCU/DSP_SDRAM_CS -> (no net)
- U1 pad 19: /MCU/DSP_SDRAM_ADRESS_BUS11 -> (no net)
- U1 pad 2: /MCU/DSP_SDRAM_DATA_BUS0 -> (no net)
- U1 pad 20: /MCU/DSP_SDRAM_ADRESS_BUS10 -> (no net)
- U1 pad 21: /MCU/DSP_SDRAM_ADRESS_BUS0 -> (no net)
- U1 pad 22: /MCU/DSP_SDRAM_ADRESS_BUS1 -> (no net)
- U1 pad 23: /MCU/DSP_SDRAM_ADRESS_BUS2 -> (no net)
- U1 pad 24: /MCU/DSP_SDRAM_ADRESS_BUS3 -> (no net)
- U1 pad 26: GND -> Audio_Loop3_Return
- U1 pad 27: /MCU/DSP_SDRAM_ADRESS_BUS4 -> (no net)
- U1 pad 28: /MCU/DSP_SDRAM_ADRESS_BUS5 -> (no net)
- U1 pad 29: /MCU/DSP_SDRAM_ADRESS_BUS6 -> (no net)
- U1 pad 3: /MCU/DSP_SDRAM_DATA_BUS1 -> (no net)
- U1 pad 30: /MCU/DSP_SDRAM_ADRESS_BUS7 -> (no net)
- U1 pad 31: /MCU/DSP_SDRAM_ADRESS_BUS8 -> (no net)
- U1 pad 32: /MCU/DSP_SDRAM_ADRESS_BUS9 -> (no net)
- U1 pad 34: /MCU/DSP_SDRAM_CKE -> (no net)
- U1 pad 35: /MCU/DSP_SDRAM_CLK -> (no net)
- U1 pad 36: /MCU/DSP_SDRAM_UDQM -> (no net)
- U1 pad 39: /MCU/DSP_SDRAM_DATA_BUS8 -> (no net)
- U1 pad 4: GND -> Audio_Loop3_Return
- U1 pad 40: /MCU/DSP_SDRAM_DATA_BUS9 -> (no net)
- U1 pad 41: GND -> Audio_Loop3_Return
- U1 pad 42: /MCU/DSP_SDRAM_DATA_BUS10 -> (no net)
- U1 pad 43: /MCU/DSP_SDRAM_DATA_BUS11 -> (no net)
- U1 pad 45: /MCU/DSP_SDRAM_DATA_BUS12 -> (no net)
- U1 pad 46: /MCU/DSP_SDRAM_DATA_BUS13 -> (no net)
- U1 pad 47: GND -> Audio_Loop3_Return
- U1 pad 48: /MCU/DSP_SDRAM_DATA_BUS14 -> (no net)
- U1 pad 49: /MCU/DSP_SDRAM_DATA_BUS15 -> (no net)
- U1 pad 5: /MCU/DSP_SDRAM_DATA_BUS2 -> (no net)
- U1 pad 50: GND -> Audio_Loop3_Return
- U1 pad 6: /MCU/DSP_SDRAM_DATA_BUS3 -> (no net)
- U1 pad 8: /MCU/DSP_SDRAM_DATA_BUS4 -> (no net)
- U1 pad 9: /MCU/DSP_SDRAM_DATA_BUS5 -> (no net)
- U11 pad 1: GND -> Audio_Loop3_Return
- U11 pad 10: DAC4P -> (no net)
- U11 pad 11: DAC4N -> (no net)
- U11 pad 12: DAC3P -> (no net)
- U11 pad 13: DAC3N -> (no net)
- U11 pad 14: +3.3V -> (no net)
- U11 pad 15: unconnected-(U11A-DSDATA4-Pad15) -> (no net)
- U11 pad 16: GND -> Audio_Loop3_Return
- U11 pad 18: unconnected-(U11A-DADATA3-Pad18) -> (no net)
- U11 pad 19: unconnected-(U11A-DSDATA2-Pad19) -> (no net)
- U11 pad 2: AD1939_MCLKI -> (no net)
- U11 pad 20: AD1939_SAI1A_SDO -> (no net)
- U11 pad 21: AD1939_SAI1A_CK -> (no net)
- U11 pad 22: AD1939_SAI1A_WS -> (no net)
- U11 pad 23: GND -> Audio_Loop3_Return
- U11 pad 24: GND -> Audio_Loop3_Return
- U11 pad 25: GND -> Audio_Loop3_Return
- U11 pad 26: unconnected-(U11A-ASDATA2-Pad26) -> (no net)
- U11 pad 27: AD1939_SAI1B_SDI -> (no net)
- U11 pad 28: AD1939_SAI1A_CK -> (no net)
- U11 pad 29: AD1939_SAI1A_WS -> (no net)
- U11 pad 3: AD1939_MCLKO -> (no net)
- U11 pad 30: AD1939_SPI_MOSI -> (no net)
- U11 pad 31: AD1939_SPI_MISO -> (no net)
- U11 pad 33: GND -> Audio_Loop3_Return
- U11 pad 34: AD1939_SPI_CLK -> (no net)
- U11 pad 35: AD1939_SPI_CS -> (no net)
- U11 pad 36: unconnected-(U11A-OL1P-Pad36) -> (no net)
- U11 pad 37: unconnected-(U11A-OL1N-Pad37) -> (no net)
- U11 pad 38: unconnected-(U11A-OR1P-Pad38) -> (no net)
- U11 pad 39: unconnected-(U11A-OR1N-Pad39) -> (no net)
- U11 pad 4: GND -> Audio_Loop3_Return
- U11 pad 40: unconnected-(U11A-OL2P-Pad40) -> (no net)
- U11 pad 41: unconnected-(U11A-OL2N-Pad41) -> (no net)
- U11 pad 42: unconnected-(U11A-OR2P-Pad42) -> (no net)
- U11 pad 43: unconnected-(U11A-OR2N-Pad43) -> (no net)
- U11 pad 44: GND -> Audio_Loop3_Return
- U11 pad 46: GND -> Audio_Loop3_Return
- U11 pad 47: AD1939_FILTR -> (no net)
- U11 pad 48: GND -> Audio_Loop3_Return
- U11 pad 52: AD1939_CM -> (no net)
- U11 pad 53: ADC1P -> (no net)
- U11 pad 54: ADC1N -> (no net)
- U11 pad 55: ADC2P -> (no net)
- U11 pad 56: ADC2N -> (no net)
- U11 pad 57: ADC3P -> (no net)
- U11 pad 58: ADC3N -> (no net)
- U11 pad 59: ADC4P -> (no net)
- U11 pad 6: DAC2P -> (no net)
- U11 pad 60: ADC4N -> (no net)
- U11 pad 61: AD1939_LF -> (no net)
- U11 pad 7: DAC2N -> (no net)
- U11 pad 8: DAC1P -> (no net)
- U11 pad 9: DAC1N -> (no net)
- U16 pad 2: GND -> Audio_Loop3_Return
- U16 pad 4: Net-(U19-DMU) -> DSP_USB_HS_D-
- U16 pad 6: Net-(U19-DPU) -> DSP_USB_HS_D+
- U20 pad 1: GND -> Audio_Loop3_Return
- U3 pad 1: GND -> Audio_Loop3_Return
- U5 pad 1: GND -> Audio_Loop3_Return
- U6 pad 2: GND -> Audio_Loop3_Return
- U7 pad 1: /MCU/DSP_FLASH_D2 -> unconnected-(U7-PE2-Pad1)
- U7 pad 10: /MCU/DSP_SDRAM_ADRESS_BUS0 -> Audio_Loop3_Return
- U7 pad 100: LED3_PIN -> +3.3V
- U7 pad 11: /MCU/DSP_SDRAM_ADRESS_BUS1 -> +3.3V
- U7 pad 12: /MCU/DSP_SDRAM_ADRESS_BUS2 -> OSC0
- U7 pad 13: /MCU/DSP_SDRAM_ADRESS_BUS3 -> OSC1
- U7 pad 14: /MCU/DSP_SDRAM_ADRESS_BUS4 -> NRST
- U7 pad 15: /MCU/DSP_SDRAM_ADRESS_BUS5 -> unconnected-(U7-PC0-Pad15)
- U7 pad 16: GND -> unconnected-(U7-PC1-Pad16)
- U7 pad 17: +3.3V -> unconnected-(U7-PC2_C-Pad17)
- U7 pad 18: /MCU/DSP_FLASH_D3 -> unconnected-(U7-PC3_C-Pad18)
- U7 pad 19: unconnected-(U7-PF7-Pad19) -> Audio_Loop3_Return
- U7 pad 2: AD1939_SAI1B_SDI -> unconnected-(U7-PE3-Pad2)
- U7 pad 20: /MCU/DSP_FLASH_D0 -> +3.3V
- U7 pad 21: /MCU/DSP_FLASH_D1 -> +3.3V
- U7 pad 22: /MCU/DSP_FLASH_CLK -> unconnected-(U7-PA0-Pad22)
- U7 pad 23: OSC0 -> unconnected-(U7-PA1-Pad23)
- U7 pad 24: OSC1 -> unconnected-(U7-PA2-Pad24)
- U7 pad 25: /MCU/NRST -> unconnected-(U7-PA3-Pad25)
- U7 pad 26: /MCU/DSP_SDRAM_WE -> Audio_Loop3_Return
- U7 pad 27: unconnected-(U7-PC1-Pad27) -> +3.3V
- U7 pad 28: /MCU/DSP_SDRAM_CS -> unconnected-(U7-PA4-Pad28)
- U7 pad 29: /MCU/DSP_SDRAM_CKE -> unconnected-(U7-PA5-Pad29)
- U7 pad 3: AD1939_SAI1A_WS -> unconnected-(U7-PE4-Pad3)
- U7 pad 30: +3.3V -> unconnected-(U7-PA6-Pad30)
- U7 pad 31: GND -> unconnected-(U7-PA7-Pad31)
- U7 pad 32: +3.3V -> unconnected-(U7-PC4-Pad32)
- U7 pad 33: +3.3V -> unconnected-(U7-PC5-Pad33)
- U7 pad 36: EXT_POT_ADC -> unconnected-(U7-PB2-Pad36)
- U7 pad 38: GND -> unconnected-(U7-PE8-Pad38)
- U7 pad 39: +3.3V -> unconnected-(U7-PE9-Pad39)
- U7 pad 4: AD1939_SAI1A_CK -> unconnected-(U7-PE5-Pad4)
- U7 pad 40: /MCU/DSP_SDRAM_DATA_BUS8 -> unconnected-(U7-PE10-Pad40)
- U7 pad 41: /MCU/DSP_SDRAM_DATA_BUS9 -> unconnected-(U7-PE11-Pad41)
- U7 pad 42: AD1939_SPI_MISO -> unconnected-(U7-PE12-Pad42)
- U7 pad 48: unconnected-(U7-PB2-Pad48) -> Net-(C1-Pad1)
- U7 pad 49: /MCU/DSP_SDRAM_RAS -> Audio_Loop3_Return
- U7 pad 5: AD1939_SAI1A_SDO -> unconnected-(U7-PE6-Pad5)
- U7 pad 50: /MCU/DSP_SDRAM_ADRESS_BUS6 -> +3.3V
- U7 pad 51: GND -> unconnected-(U7-PB12-Pad51)
- U7 pad 52: +3.3V -> unconnected-(U7-PB13-Pad52)
- U7 pad 53: /MCU/DSP_SDRAM_ADRESS_BUS7 -> unconnected-(U7-PB14-Pad53)
- U7 pad 54: /MCU/DSP_SDRAM_ADRESS_BUS8 -> unconnected-(U7-PB15-Pad54)
- U7 pad 55: /MCU/DSP_SDRAM_ADRESS_BUS9 -> unconnected-(U7-PD8-Pad55)
- U7 pad 56: /MCU/DSP_SDRAM_ADRESS_BUS10 -> unconnected-(U7-PD9-Pad56)
- U7 pad 58: /MCU/DSP_SDRAM_DATA_BUS4 -> unconnected-(U7-PD11-Pad58)
- U7 pad 59: /MCU/DSP_SDRAM_DATA_BUS5 -> unconnected-(U7-PD12-Pad59)
- U7 pad 60: /MCU/DSP_SDRAM_DATA_BUS6 -> unconnected-(U7-PD13-Pad60)
- U7 pad 61: GND -> unconnected-(U7-PD14-Pad61)
- U7 pad 62: +3.3V -> unconnected-(U7-PD15-Pad62)
- U7 pad 63: /MCU/DSP_SDRAM_DATA_BUS7 -> unconnected-(U7-PC6-Pad63)
- U7 pad 64: /MCU/DSP_FLASH_CS -> unconnected-(U7-PC7-Pad64)
- U7 pad 66: /MCU/DSP_SDRAM_DATA_BUS10 -> unconnected-(U7-PC9-Pad66)
- U7 pad 67: /MCU/DSP_SDRAM_DATA_BUS11 -> unconnected-(U7-PA8-Pad67)
- U7 pad 68: /MCU/DSP_SDRAM_DATA_BUS12 -> unconnected-(U7-PA9-Pad68)
- U7 pad 71: Net-(C1-Pad1) -> unconnected-(U7-PA12-Pad71)
- U7 pad 72: +3.3V -> unconnected-(U7-PA13-Pad72)
- U7 pad 73: unconnected-(U7-PB12-Pad73) -> Net-(C49-Pad1)
- U7 pad 74: unconnected-(U7-PB13-Pad74) -> Audio_Loop3_Return
- U7 pad 75: unconnected-(U7-PB14-Pad75) -> +3.3V
- U7 pad 77: /MCU/DSP_SDRAM_DATA_BUS13 -> unconnected-(U7-PA15-Pad77)
- U7 pad 78: /MCU/DSP_SDRAM_DATA_BUS14 -> unconnected-(U7-PC10-Pad78)
- U7 pad 79: /MCU/DSP_SDRAM_DATA_BUS15 -> unconnected-(U7-PC11-Pad79)
- U7 pad 81: I2C_SCL -> unconnected-(U7-PD0-Pad81)
- U7 pad 82: I2C_SDA -> unconnected-(U7-PD1-Pad82)
- U7 pad 83: GND -> unconnected-(U7-PD2-Pad83)
- U7 pad 84: +3.3V -> unconnected-(U7-PD3-Pad84)
- U7 pad 85: /MCU/DSP_SDRAM_DATA_BUS0 -> unconnected-(U7-PD4-Pad85)
- U7 pad 86: /MCU/DSP_SDRAM_DATA_BUS1 -> unconnected-(U7-PD5-Pad86)
- U7 pad 89: /MCU/DSP_SDRAM_ADRESS_BUS11 -> unconnected-(U7-PB3-Pad89)
- U7 pad 90: DSP_OK_LED -> unconnected-(U7-PB4-Pad90)
- U7 pad 93: /MCU/DSP_SDRAM_CLK -> unconnected-(U7-PB7-Pad93)
- U7 pad 94: GND -> to_BOOT0
- U7 pad 95: +3.3V -> unconnected-(U7-PB8-Pad95)
- U7 pad 99: LED4_PIN -> Audio_Loop3_Return
- U9 pad 1: GND -> unconnected-(U9-SDIN-Pad1)
- U9 pad 2: +3.3V -> unconnected-(U9-LRCLK-Pad2)
- U9 pad 3: 5V -> unconnected-(U9-MCLK-Pad3)
- U9 pad 4: (no net) -> unconnected-(U9-SCLK-Pad4)
- Y2 pad 2: GND -> Audio_Loop3_Return
- Y2 pad 4: GND -> Audio_Loop3_Return
Routing:
- net (no net): track 0.00 -> 1963.8 mm, vias 0 -> 25
- net AD1939_CM: track 257.2 -> 0.00 mm, vias 9 -> 0
- net GND: track 247.3 -> 11.6 mm, vias 929 -> 0
- net Audio_Loop3_Return: track 35.9 -> 225.1 mm, vias 0 -> 884
- net Net-(J1-PadR): track 153.1 -> 0.00 mm
- net POT3: track 138.1 -> 0.00 mm
- net DISPLAY_USB_HS_D+: track 134.5 -> 0.00 mm
- net DISPLAY_USB_HS_D-: track 134.5 -> 0.00 mm
- net POT6: track 126.7 -> 0.00 mm
- net POT2: track 97.4 -> 0.00 mm
- net POT5: track 88.2 -> 0.00 mm
- net POT1: track 67.7 -> 0.00 mm
- net POT4: track 51.7 -> 0.00 mm
- net NRST: track 0.00 -> 51.4 mm, vias 0 -> 2
- net unconnected-(U9-SDIN-Pad1): track 0.00 -> 45.7 mm, vias 0 -> 43
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- added copper zone on F.Cu, net Audio_Loop3_Return
- added copper zone on In1.Cu, net Audio_Loop3_Return
- added copper zone on In2.Cu, net Audio_Loop3_Return
- removed copper zone on F.Cu, net GND
- removed copper zone on In1.Cu, net GND
- removed copper zone on In2.Cu, net GND
