File: sab_v4_mini/Input_stage.kicad_sch (KiCad schematic)
At the start: 92 parts, among them U4 OP275

Commit message: moved codec
Parts:
- removed C17 (x2): 1p, Capacitor_SMD:C_0603_1608Metric, symbol Device:C_Small
- removed C18 (x8): 100nF, Capacitor_SMD:C_0603_1608Metric, symbol Device:C_Small
- removed C18 (x2), C19 (x4), C24 (x4): 100pF, Capacitor_SMD:C_0603_1608Metric, symbol Device:C_Small
- removed C21 (x2), C23 (x4): 1nF, Capacitor_SMD:C_0603_1608Metric, symbol Device:C_Small
- removed D1, D12, D13, D14, D15, D16, D19, D20, D4, D7, D8, D9: 1N5819, Diode_SMD:D_SOD-323, symbol Diode:1N5819
- removed R4 (x8), R8 (x2), R9 (x4): 100R, Resistor_SMD:R_0603_1608Metric, symbol Device:R
- removed R4 (x2): 1M, Resistor_SMD:R_0603_1608Metric, symbol Device:R
- removed R5 (x2): 510k, Resistor_SMD:R_0603_1608Metric, symbol Device:R
- removed R6 (x4), R7 (x4): 4k7, Resistor_SMD:R_0603_1608Metric, symbol Device:R
- removed unit 2 of U4 (x4)
Connections:
- net ADC1N renamed CS4270_ANALOG_IN_A
- net ADC3N renamed CS4270_ANALOG_IN_B
- net Audio_Loop1_Return renamed AUDIO_IN_B
- net Audio_Loop3_Return renamed AUDIO_IN_A
Other:
- moved on the sheet: C18, C21, D17, D18, D5, D6, R4, R8
